File: krokowka-driver/SterownikCNC4.sch (EAGLE design)
At the start: 55 parts, among them IC1 NC7WP14P6X, IC4 NC7WP14P6X, T2 N_MOSFET-TO263, T3 N_MOSFET-TO263, T4 N_MOSFET-TO263, T5 N_MOSFET-TO263, T6 N_MOSFET-TO263, T7 N_MOSFET-TO263, T8 N_MOSFET-TO263, T9 N_MOSFET-TO263

Commit message: added krokowka-driver/
Parts:
- removed IC2: (no value), v-reg-3:LM1117
- added IC3: NC7WP14P6X, bufory,invertery:NC7WP14P6X
- added U$6: TS9011SCX, v-reg:TS9011SCX
Connections:
- net +3V3: now also U$6.OUT; no longer IC2.OUT
- net GND: now also U$6.GND; no longer IC2.GND
- net PWM2: now also IC3G$1.I; no longer IC4G$1.I
- net PWM2_NEG: now also IC3G$1.O; no longer IC4G$1.O
- net VCC: now also U$6.IN; no longer IC2.IN

Commit message: Add existing file
Parts:
- removed T2, T3, T4, T5, T6, T7, T8, T9: N_MOSFET-TO263, robione:N_MOSFET-TO263
- added Q1, Q2, Q3, Q4, Q5, Q6, Q7, Q8: IRF3704S, transistor-power:IRF3704S
- added U$7, U$9: PTB-02_5.08MM, robione:PTB-02_5.08MM
Connections:
- net +24V: now also Q1.D, Q3.D, Q6.D, Q8.D; no longer T2.D, T4.D, T6.D, T8.D
- net GNDA: now also Q2.S, Q4.S, Q5.S, Q7.S; no longer T3.S, T5.S, T7.S, T9.S
- net M_OUT: now also Q1.S, Q2.D, U$7.1; no longer T2.S, T3.D
- net M_OUT1: now also Q7.D, Q8.S, U$7.2; no longer T6.S, T7.D
- net M_OUT2: now also Q3.S, Q4.D, U$9.1; no longer T4.S, T5.D
- net M_OUT3: now also Q5.D, Q6.S, U$9.2; no longer T8.S, T9.D
- net N$1: now also Q1.G; no longer T2.G
- net N$10: now also Q7.G; no longer T7.G
- net N$11: now also Q8.G; no longer T6.G
- net N$16: now also Q4.G; no longer T5.G
- net N$17: now also Q3.G; no longer T4.G
- net N$2: now also Q2.G; no longer T3.G
- net N$22: now also Q5.G; no longer T9.G
- net N$23: now also Q6.G; no longer T8.G
Other:
- note added: "Trzeba przetestowac"
- note added: "Wtyki silników"
