File: krokowka-driver/SterownikCNC4.sch (EAGLE design)
At the start: 57 parts, among them IC1 NC7WP14P6X, IC4 NC7WP14P6X, Q1 IRF3704S, Q2 IRF3704S, Q3 IRF3704S, Q4 IRF3704S, Q5 IRF3704S, Q6 IRF3704S, Q7 IRF3704S, Q8 IRF3704S, U1 IR2104, U2 IR2104, U3 IR2104, U4 IR2104

Commit message: zmina_30.12
Parts:
- removed C5: 1uF/50v, rcl:C-EUC0603K
- C9: value 100uF/63V -> 100uF; device rcl:CPOL-EUE5-10.5 -> rcl:CPOL-EU153CLV-0810
Connections:
- removed net +12V: C11.1, C13.1, C14.1, C7.1, D4.A, D5.A, D6.A, D7.A, U1.VCC, U2.VCC, U3.VCC, U4.VCC
- net +24V: no longer C5.1, C9.+
- net GNDA: no longer C5.2
- net N$13: now also C9.+
- net VCC: now also C11.1, C13.1, C14.1, C7.1, D4.A, D5.A, D6.A, D7.A, U1.VCC, U2.VCC, U3.VCC, U4.VCC
Other:
- moved on the sheet: C9, D1, F1
