File: krokowka-driver/SterownikCNC4_1.brd (EAGLE design)
At the start: 60.6 x 45.7 mm, 56 parts, among them IC1 NC7WP14P6X, IC4 NC7WP14P6X, Q1 IRF3704S, Q2 IRF3704S, Q3 IRF3704S, Q4 IRF3704S, Q5 IRF3704S, Q6 IRF3704S, Q7 IRF3704S, Q8 IRF3704S, U1 IR2104, U2 IR2104, U3 IR2104, U4 IR2104

Commit message: Nowa wersja, eagle cos zjebal
Parts:
- moved D7 9.67 mm to (54.6, 4.47), turned to 0 degrees
- moved IC4 6.35 mm to (40.6, 7.62)
- moved C14 4.26 mm to (53.1, 6.53), turned to 0 degrees
- moved U$2 1.27 mm to (53.3, 3.81)
- moved C9 1.07 mm to (44.2, 5.99)
- moved C13 0.76 mm to (26.6, 10.5), turned to 90 degrees
- moved C7 0.73 mm to (11.3, 10.5), turned to 90 degrees
- moved C11 0.63 mm to (42.0, 10.5), turned to 90 degrees
- moved D3 0.36 mm to (33.0, 5.99)
- moved C15 0.28 mm to (55.5, 14.9)
Routing:
- net GND: track 126.7 -> 48.2 mm, vias 9 -> 3
- net N$18: track 4.81 -> 18.6 mm
- net +3V3: track 52.2 -> 38.6 mm
- net VCC: track 83.5 -> 91.4 mm, vias 1 -> 2
- net PWM2_NEG: track 12.7 -> 4.82 mm
- net N$6: track 6.16 -> 13.5 mm
- net N$13: track 20.3 -> 22.5 mm
- net PWM1: track 27.8 -> 26.1 mm
- net M_OUT: track 68.4 -> 66.9 mm
- net M_OUT2: track 66.5 -> 65.1 mm
- net M_OUT1: track 59.2 -> 58.2 mm
- net N$5: track 8.31 -> 7.40 mm
- net M_OUT3: track 60.0 -> 59.2 mm
- net PWM2: track 25.7 -> 24.9 mm
- net GNDA: vias 7 -> 8
Other:
- board text added: "Dodać biblioteke zlacz silnika"
- board text added: "Napisy w bibliotece t-deans"
- board text added: "To Do:"
- board text removed: "Logika i zasilanie 12v do wyplatania"
- board text removed: "Napisy do poprawienia"
- board text removed: "Pamietac o ERC 8mils"
