File: krokowka-driver/SterownikDriver_01.sch (EAGLE design)
At the start: 56 parts, among them IC1 NC7WP14P6X, IC4 NC7WP14P6X, Q1 IRF3704S, Q2 IRF3704S, Q3 IRF3704S, Q4 IRF3704S, Q5 IRF3704S, Q6 IRF3704S, Q7 IRF3704S, Q8 IRF3704S, U1 IR2104, U2 IR2104, U3 IR2104, U4 IR2104

Commit message: ver 0.2
Parts:
- removed IC4: NC7WP14P6X, bufory,invertery:NC7WP14P6X
- added R10, R9: 10, rcl:R-EU_R0603
Connections:
- removed net N$5: IC1G$2.O, U2.PWM
- removed net N$6: IC4G$2.O, U4.PWM
- net +3V3: no longer IC4G$3.VCC
- net GND: now also R10.1, R9.1; no longer IC4G$3.GND
- net PWM1: now also IC1G$2.I, R10.2, U2.PWM; no longer IC1G$1.I
- net PWM1_NEG: now also IC1G$2.O; no longer IC1G$1.O, IC1G$2.I
- net PWM2: now also IC1G$1.I, R9.2, U4.PWM; no longer IC4G$1.I
- net PWM2_NEG: now also IC1G$1.O; no longer IC4G$1.O, IC4G$2.I
Other:
- note removed: "Wstepnie gold-piny"
