File: glowna/glowna.sch (EAGLE design)
At the start: 30 parts

Commit message: ferryt
Connections:
- removed net N$7: U$1.VDDA, U$1.VREF+, U$2.2
- new net N$5: C3.1, C4.1, U$1.VDDA, U$1.VDD_0, U$1.VREF+, U$2.2
- net +3V3: no longer C3.1, C4.1, U$1.VDD_0
Changed lines of the file:
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@@
 <instance part="C16" gate="G$1" x="-35.56" y="109.22" rot="R180"/>
 <instance part="S1" gate="G$1" x="-35.56" y="20.32"/>
-<instance part="U$2" gate="G$1" x="-7.62" y="10.16" smashed="yes" rot="R90">
-<attribute name="VALUE" x="-1.27" y="13.462" size="1.778" layer="96" rot="R180"/>
+<instance part="U$2" gate="G$1" x="-35.56" y="0" smashed="yes" rot="R90">
+<attribute name="VALUE" x="-29.21" y="3.302" size="1.778" layer="96" rot="R180"/>
 </instance>
 <instance part="+3V1" gate="G$1" x="-35.56" y="119.38" smashed="yes">
@@
 <attribute name="VALUE" x="25.4" y="-35.56" size="1.778" layer="96" rot="R180"/>
 </instance>
-<instance part="+3V12" gate="G$1" x="-20.32" y="20.32" smashed="yes">
-<attribute name="VALUE" x="-17.78" y="22.86" size="1.778" layer="96" rot="R180"/>
+<instance part="+3V12" gate="G$1" x="-43.18" y="5.08" smashed="yes">
+<attribute name="VALUE" x="-40.64" y="7.62" size="1.778" layer="96" rot="R180"/>
 </instance>
 <instance part="R2" gate="G$1" x="-27.94" y="35.56" smashed="yes" rot="R270">
@@
 </segment>
 </net>
-<net name="N$7" class="0">
-<segment>
-<pinref part="U$2" gate="G$1" pin="2"/>
-<pinref part="U$1" gate="G$1" pin="VREF+"/>
-<wire x1="-2.54" y1="10.16" x2="0" y2="10.16" width="0.1524" layer="91"/>
-<pinref part="U$1" gate="G$1" pin="VDDA"/>
-<wire x1="0" y1="10.16" x2="2.54" y2="10.16" width="0.1524" layer="91"/>
-<wire x1="2.54" y1="7.62" x2="0" y2="7.62" width="0.1524" layer="91"/>
-<wire x1="0" y1="7.62" x2="0" y2="10.16" width="0.1524" layer="91"/>
-<junction x="0" y="10.16"/>
-</segment>
-</net>
 <net name="+3V3" class="0">
 <segment>
@@
 </segment>
 <segment>
-<pinref part="U$1" gate="G$1" pin="VDD_0"/>
-<wire x1="2.54" y1="15.24" x2="-20.32" y2="15.24" width="0.1524" layer="91"/>
-<wire x1="-20.32" y1="15.24" x2="-20.32" y2="17.78" width="0.1524" layer="91"/>
-<wire x1="-20.32" y1="10.16" x2="-20.32" y2="15.24" width="0.1524" layer="91"/>
-<junction x="-20.32" y="15.24"/>
-<wire x1="-20.32" y1="7.62" x2="-20.32" y2="10.16" width="0.1524" layer="91"/>
-<junction x="-20.32" y="10.16"/>
-<pinref part="C3" gate="G$1" pin="1"/>
-<pinref part="C4" gate="G$1" pin="1"/>
-<wire x1="-25.4" y1="7.62" x2="-25.4" y2="10.16" width="0.1524" layer="91"/>
-<wire x1="-25.4" y1="10.16" x2="-20.32" y2="10.16" width="0.1524" layer="91"/>
-<wire x1="-20.32" y1="10.16" x2="-12.7" y2="10.16" width="0.1524" layer="91"/>
-<pinref part="U$2" gate="G$1" pin="1"/>
-<pinref part="+3V12" gate="G$1" pin="+3V3"/>
-</segment>
-<segment>
 <pinref part="R2" gate="G$1" pin="1"/>
 <pinref part="+3V13" gate="G$1" pin="+3V3"/>
@@
 <pinref part="+3V16" gate="G$1" pin="+3V3"/>
 <wire x1="-162.56" y1="99.06" x2="-162.56" y2="96.52" width="0.1524" layer="91"/>
+</segment>
+<segment>
+<pinref part="+3V12" gate="G$1" pin="+3V3"/>
+<wire x1="-43.18" y1="2.54" x2="-43.18" y2="0" width="0.1524" layer="91"/>
+<pinref part="U$2" gate="G$1" pin="1"/>
+<wire x1="-43.18" y1="0" x2="-40.64" y2="0" width="0.1524" layer="91"/>
 </segment>
 </net>
@@
 </segment>
 </net>
+<net name="N$5" class="0">
+<segment>
+<pinref part="U$1" gate="G$1" pin="VDD_0"/>
+<wire x1="2.54" y1="15.24" x2="-20.32" y2="15.24" width="0.1524" layer="91"/>
+<wire x1="-20.32" y1="10.16" x2="-20.32" y2="15.24" width="0.1524" layer="91"/>
+<wire x1="-20.32" y1="7.62" x2="-20.32" y2="10.16" width="0.1524" layer="91"/>
+<junction x="-20.32" y="10.16"/>
+<pinref part="C3" gate="G$1" pin="1"/>
+<pinref part="C4" gate="G$1" pin="1"/>
+<wire x1="-25.4" y1="7.62" x2="-25.4" y2="10.16" width="0.1524" layer="91"/>
+<wire x1="-25.4" y1="10.16" x2="-20.32" y2="10.16" width="0.1524" layer="91"/>
+<pinref part="U$1" gate="G$1" pin="VREF+"/>
+<pinref part="U$1" gate="G$1" pin="VDDA"/>
+<wire x1="0" y1="10.16" x2="2.54" y2="10.16" width="0.1524" layer="91"/>
+<wire x1="2.54" y1="7.62" x2="0" y2="7.62" width="0.1524" layer="91"/>
+<wire x1="0" y1="7.62" x2="0" y2="10.16" width="0.1524" layer="91"/>
+<wire x1="-20.32" y1="10.16" x2="0" y2="10.16" width="0.1524" layer="91"/>
+<junction x="0" y="10.16"/>
+<pinref part="U$2" gate="G$1" pin="2"/>
+<wire x1="-25.4" y1="7.62" x2="-30.48" y2="7.62" width="0.1524" layer="91"/>
+<wire x1="-30.48" y1="7.62" x2="-30.48" y2="0" width="0.1524" layer="91"/>
+<junction x="-25.4" y="7.62"/>
+</segment>
+</net>

Commit message: glowna
Parts:
- added C18, C19: 20pF?, rcl:C-EUC0603
- added D1, D2, D3: (no value), diode:DIODE-DO-214AC
- added DRIVERS, HEATERS, LOGIC: (no value), pinhead:PINHD-1X2
- added JP1, JP2, JP3, JP4, JP5, JP6: (no value), pinhead:PINHD-1X4
- added Q1: CSM-7X-DU, crystal:CSM-7X-DU
- added U$10, U$11, U$12, U$13, U$14, U$15, U$16, U$17, U$18, U$7, U$8, U$9: T-DEANS, Conector_T-deans:T-DEANS
- added X2: MINI-USB_SHIELD4P-32005-101, con-cypressindustries:MINI-USB_SHIELD4P-32005-101
- R3: value 10k -> 1.5k
Connections:
- removed net N$11: U$5.E
- removed net TIM_5PWM_Y3: U$1.PA2
- new net +12V: D1.C, JP1.1, JP2.1, JP3.1, JP5.1, JP6.1, LOGIC.1, U$5.E
- new net +24V: D2.C, D3.C, DRIVERS.1, HEATERS.1, U$11.P$1, U$11.P$2, U$13.P$1, U$13.P$2, U$15.P$1, U$15.P$2, U$17.P$1, U$17.P$2, U$7.P$1, U$7.P$2, U$9.P$1, U$9.P$2
- new net RCC_IN: C18.2, Q1.2, U$1.PH0
- new net RCC_OUT: C19.2, Q1.1, U$1.PH1
- new net TIM5_PWM_Y3: JP2.4, U$1.PA2
- net GND: now also C18.1, C19.1, D1.A, D2.A, D3.A, DRIVERS.2, HEATERS.2, LOGIC.2, U$10.P$1, U$10.P$2, U$12.P$1, U$12.P$2, U$14.P$1, U$14.P$2, U$16.P$1, U$16.P$2, U$18.P$1, U$18.P$2, U$8.P$1, U$8.P$2
- net TIM12_EX2_1: now also JP5.3
- net TIM12_EX2_2: now also JP5.4
- net TIM4_PWM_X1: now also JP1.2
- net TIM4_PWM_X2: now also JP1.3
- net TIM4_PWM_X3: now also JP1.4
- net TIM5_EX1_1: now also JP4.3
- net TIM5_PWM_Y1: now also JP2.2
- net TIM5_PWM_Y2: now also JP2.3
- net TIM8_EX1_2: now also JP4.4
- net TIM8_PWM_Z1: now also JP3.2
- net TIM8_PWM_Z2: now also JP3.3
- net TIM8_PWM_Z3: now also JP3.4
- net TIM9_EX3_1: now also JP6.3
- net TIM9_EX3_2: now also JP6.4
Other:
- note added: "Boże, daj mi siłe bym znalazł cokolwiek mniej chujowego niż to"
- note added: "Chciałbym się przypierdolić... ale nie mam lepszego pomysłu"
- note added: "Co robimy z rs485?"
- note added: "Filtrujemy czy jebac?"
- note added: "Jaki kwarc?"
- note added: "Jakie złącza ?"
- note added: "Jest miejsce to napisz anime jakieś fajne bo tamto już kończę"
- note added: "Mosfety do sterowania w jakiej obudowie?"
- note added: "Offtopic"
- note added: "Piter, znajdz scalak pod 3.3 albo CAN"
- note added: "Rs485/CAN"
- note added: "Tu leci tlyko PWM"
- note added: "USB mini B?"
- note added: "Wtyczka pierwsza ma dziwnie zrealizowane pwm, zostawiamy?"
- note added: "Wyliczymy jak już będzie dobrany kwarc"
- note added: "Zasady: 1. GND dol, VCC gora, reszta wmiare logicznie 2. Zmiany komentujemy na fioletowo 3. Biblioteki do kazdego elementu w folderze 4. "Zrobić tak by działało""
- note added: "Zlacza ADC"
- note added: "Zlacza Enkodery"
- note added: "Zlacze Wentylatory"
- note added: "Złacze LASER"
- note added: "Złącza grzałki"
- note added: "Złącza silniki"
- note added: "może jakiś elektrolit ?"
- moved on the sheet: C16, R3, R4, R5, R6, U$4, U$5, U$6
