File: glowna/plyta_glowna0.1.brd (EAGLE design)
At the start: 100 x 80 mm, 227 parts, among them IC1 4504D, IC2 MAX481CSA, IC3 4504D, IC4 OPA4658UU, Q1 CSM-7X-DU, Q2 N-HEXFET-2D_SOT232-IRLL014N, Q3 N-HEXFET-2D_SOT232-IRLL014N

Commit message: 5v enkoder
Parts:
- removed C36, C37, C38, C39: 10nF, rcl:C0603
- removed D21, D22, D23, D24, D25, D26: BAT54S, diode:SOT23
- added U$26: TS9011SCX, v-reg:SOT23
- C34: value 10nF -> 1uF
- C35: value 10nF -> 100nF
- moved C35 283.1 mm to (-167.6, -125.7)
- moved C34 282.5 mm to (-160.0, -125.7)
Connections:
- new net N$99: C34.2, JP10.1, JP11.1, JP12.1, U$26.2
- net +12V: now also C35.2, U$26.3; no longer JP10.1, JP11.1, JP12.1
- net +3V3: no longer D21.2, D22.2, D23.2, D24.2, D25.2, D26.2
- net GND: now also U$26.1; no longer C36.1, C37.1, C38.1, C39.1, D21.1, D22.1, D23.1, D24.1, D25.1, D26.1
- net TIM1_ENKODER1: no longer C34.2, D21.3
- net TIM1_ENKODER2: no longer C35.2, D22.3
- net TIM2_ENKODER1: no longer C38.2, D25.3
- net TIM2_ENKODER2: no longer C39.2, D26.3
- net TIM3_ENKODER1: no longer C36.2, D23.3
- net TIM3_ENKODER2: no longer C37.2, D24.3

Commit message: ver 0.2
Parts:
- removed F2: FUSESH22,5A, fuse:SH22,5A
- removed F3: (no value), fuse:SH32
- removed GRZALKA: (no value), pinhead:1X02
- removed R12, R16: 300, rcl:R0603
- removed R3: 1.5k, rcl:R0603
- removed R81: 1k, rcl:R0603
- removed U$5: PNP-SOT223, robione:SOT223
- removed U$6: TS9011SCX, v-reg:SOT23
- added F4, F5: FUSEBLANK_5X20MM, fuse:FUSE_HOLDER_5X20MM
- added GRZALKA4: (no value), pinhead:1X02
- added IC5: LM340H-05, linear:TO220H
- added X1: KUSBVX-BS1N, con-kycon:KUSBVX-BS1N
- C18, C19: value 20pF? -> 30pF
- C31: value 10\uF -> 100uF
- Q1: value CSM-7X-DU -> (none); device crystal:CSM-7X-DU -> crystal:HC49UP
- R82: value 1k -> 120
- moved R38 314.5 mm to (-182.9, -156.2)
- moved R11 312.1 mm to (-182.9, -130.8)
- moved R35 311.8 mm to (-182.9, -146.1)
- moved R42 302.2 mm to (-182.9, -151.1)
- moved R29 272.5 mm to (-182.9, -141.0)
- moved R28 268.5 mm to (-182.9, -135.9)
- moved Q1 255.5 mm to (-177.8, -163.8)
- moved GRZALKA1 33.0 mm to (-123.2, 97.8)
- moved GRZALKA2 11.4 mm to (-90.2, 97.8)
- renumbered JP1 to M1, JP10 to ENKODER2, JP11 to ENKODER1, JP12 to ENKODER3, JP13 to ADC1, JP14 to ADC2, JP15 to ADC3, JP16 to ADC4, JP17 to KR1, JP18 to KR2, JP19 to KR3, JP2 to M2, JP20 to KR4, JP21 to KR5, JP22 to KR6, JP23 to RS-485, JP24 to KR7, JP25 to I2C, JP26 to WIFI, JP27 to INDUKCYJNY, JP3 to M3, JP4 to M6, JP5 to M5, JP6 to M4, JP7 to LASER, JP8 to WEN1, JP9 to WEN2, SV1 to LCD1, SV2 to LCD2, U$10 to M2-, U$11 to M3+, U$12 to M3-, U$13 to M6+, U$14 to M6-, U$15 to M5+, U$16 to M5-, U$17 to M4+, U$18 to M4-, U$19 to V-RS, U$26 to V-ENK, U$7 to M1+, U$8 to M1-, U$9 to M2+
Connections:
- removed net N$1: R3.1, U$5.1
- removed net N$16: C29.2, IC1.1, R12.1
- removed net N$39: C30.2, IC1.16, R16.1
- removed net N$4: R3.2, U$6.3
- removed net N$66: R81.1, RS-485.1
- removed net N$82: R82.1, RS-485.2
- net +12V: now also C30.1, IC1.16, IC5.1; no longer R16.2, U$5.3
- net +24V: now also F4.2; no longer F3.2A
- net +3V3: now also C29.2, IC1.1, IC5.3, X1.1; no longer R12.2, U$5.2, U$5.4, U$6.2
- net GND: now also ADC2.1, ADC3.1, ADC4.1, C30.2, IC5.2, R11.1, X1.4; no longer C30.1, R11.2, U$6.1
- net N$10: now also F5.1; no longer F2.1
- net N$12: now also GRZALKA1.1; no longer GRZALKA.1
- net N$13: now also X1.2
- net N$14: now also X1.3
- net N$17: now also GRZALKA2.1; no longer GRZALKA1.1
- net N$18: now also GRZALKA4.1; no longer GRZALKA2.1
- net N$30: now also R82.1, RS-485.1; no longer R81.2
- net N$31: now also RS-485.2
- net N$52: now also R29.2; no longer R28.2
- net N$53: now also R28.2; no longer R29.2
- net N$8: now also F4.1; no longer F3.1A
- net N$96: now also R11.2; no longer R11.1
- net TIM8_PWM_Z2: now also R28.1; no longer R29.1
- net TIM8_PWM_Z3: now also R29.1; no longer R28.1
- net VDD: now also F5.2, GRZALKA4.2; no longer F2.2, GRZALKA.2

Commit message: Complete Ver 0.1
Parts:
- removed C40, C43, C45: 5nF, rcl:C0603
- removed IC5: LM340H-05, linear:TO220H
- removed M1+, M1-, M2+, M2-, M3+, M3-, M4+, M4-, M5+, M5-, M6+, M6-: T-DEANS, Conector_T-deans:T-DEANS
- removed Q1: (no value), crystal:HC49UP
- added 1, 10, 11, 12, 2, 3, 4, 5, 6, 7, 8, 9: PLYTKA_T, Conector_T-deans:PLYTKA_T
- added 4,7UH: FERYT_0603, rcl:R0603
- added C36: 10nF, rcl:C0603
- added C37: 100nF, rcl:C0603
- added JP1: (no value), pinhead:1X04
- added R12: 16.3k, rcl:R0603
- added R3: 49.9k, rcl:R0603
- added SHOTKY1: (no value), diode:DO-214AC
- added U$5: AP3211, Przetwornice:TSOT23
- added U$6: USBLC6-2, ESD_protection:SOT95P275X110-6N
- added XTAL1: 7M-16.000MAAJ-T, TXC-7M-16.000MAAJ-T:TXC_7M-16.000MAAJ-T
- C27: value 50nF -> 100nF
- C28: value 1uF -> 100nF
- C31: value 100uF -> 10uF; device rcl:UD-8X10_NICHICON -> rcl:C0603
- C32: value 100nF -> 22uF
- moved F5 354.3 mm to (15.2, 105.4)
- moved X1 337.7 mm to (64.8, 114.3)
- moved F4 275.7 mm to (16.5, 16.5)
- moved C7 210.9 mm to (71.1, 45.7), turned to 90 degrees
- moved C11 209.8 mm to (82.5, 69.8)
- moved C8 204.9 mm to (77.5, 48.3), turned to 270 degrees
- moved C6 198.8 mm to (66.0, 45.7), turned to 90 degrees
- moved C5 185.7 mm to (59.7, 45.7), turned to 90 degrees
- moved C16 184.2 mm to (50.8, 73.7)
- moved C1 182.4 mm to (80.0, 48.3), turned to 270 degrees
- moved C3 165.1 mm to (48.3, 53.3), turned to 270 degrees
- moved C2 150.9 mm to (40.6, 53.3), turned to 270 degrees
- moved R1 145.0 mm to (57.1, 78.7)
- moved U$2 141.6 mm to (45.7, 53.3), turned to 90 degrees
- moved C19 138.0 mm to (45.7, 57.1), turned to 180 degrees
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Connections:
- removed net N$14: R15.2, X1.3
- new net N$1: 4,7UH.1, C36.1, SHOTKY1.C, U$5.6
- new net N$16: U$6.1, X1.3
- new net N$39: C36.2, U$5.1
- new net N$4: R14.2, U$6.6
- new net NRST: C2.1, JP1.4, R2.2, S1.3, S1.4, U$1.25
- net +12V: now also C31.2, U$5.2, U$5.5; no longer IC5.1
- net +24V: now also 1.P$2, 1.P$3, 1.P$4, 1.P$5, 11.P$2, 11.P$3, 11.P$4, 11.P$5, 3.P$2, 3.P$3, 3.P$4, 3.P$5, 5.P$2, 5.P$3, 5.P$4, 5.P$5, 7.P$2, 7.P$3, 7.P$4, 7.P$5, 9.P$2, 9.P$3, 9.P$4, 9.P$5; no longer M1+.P$1, M1+.P$2, M1+.P$3, M2+.P$1, M2+.P$2, M2+.P$3, M3+.P$1, M3+.P$2, M3+.P$3, M4+.P$1, M4+.P$2, M4+.P$3, M5+.P$1, M5+.P$2, M5+.P$3, M6+.P$1, M6+.P$2, M6+.P$3
- net +3V3: now also 4,7UH.2, C37.1, R3.1, U$6.5; no longer C31.+, IC5.3, X1.1
- net GND: now also 10.P$2, 10.P$3, 10.P$4, 10.P$5, 12.P$2, 12.P$3, 12.P$4, 12.P$5, 8.P$2, 8.P$3, 8.P$4, 8.P$5, C31.1, C37.2, JP1.2, R12.2, SHOTKY1.A, U$5.4, U$6.2; no longer C31.-, IC5.2, M4-.P$1, M4-.P$2, M4-.P$3, M5-.P$1, M5-.P$2, M5-.P$3, M6-.P$1, M6-.P$2, M6-.P$3
- net N$13: now also R15.2, U$6.4; no longer R14.2, X1.2
- net N$3: now also R12.1, R3.2, U$5.3; no longer C2.1, R2.2, S1.3, S1.4, U$1.25
- net N$54: now also U$6.3, X1.2; no longer R30.1
- net N$73: no longer C40.1
- net N$75: no longer C40.2
- net N$76: no longer C45.2
- net N$77: now also 2.P$2, 2.P$3, 2.P$4, 2.P$5; no longer M1-.P$1, M1-.P$2, M1-.P$3
- net N$78: now also 4.P$2, 4.P$3, 4.P$4, 4.P$5; no longer M2-.P$1, M2-.P$2, M2-.P$3
- net N$79: no longer C45.1
- net N$80: no longer C43.2
- net N$81: no longer C43.1
- net N$83: now also 6.P$2, 6.P$3, 6.P$4, 6.P$5; no longer M3-.P$1, M3-.P$2, M3-.P$3
- net RCC_IN: now also XTAL1.3; no longer Q1.2
- net RCC_OUT: now also XTAL1.1; no longer Q1.1
- net SWCLK: now also JP1.1
- net SWDIO: now also JP1.3
- net TIM8_PWM_Z1: now also R30.1
Routing:
- net NRST: track 0.00 -> 72.6 mm, vias 0 -> 2
- net +3V3: track 0.00 -> 53.5 mm
- net SWDIO: track 0.00 -> 23.9 mm, vias 0 -> 1
- net RCC_OUT: track 0.00 -> 15.7 mm
- net N$5: track 0.00 -> 13.6 mm
- net RCC_IN: track 0.00 -> 13.4 mm
- net SWCLK: track 0.00 -> 12.7 mm
- net N$26: track 0.00 -> 8.37 mm
- net GND: track 0.00 -> 4.58 mm
- net N$19: track 0.00 -> 3.84 mm
- net N$2: track 0.00 -> 3.81 mm
- added copper zone on layer 1, net GND
Other:
- board size 100 x 80 mm -> 168.6 x 129.5 mm
